File: Embedded Systems Hardware Design/Project_HC/P2_uController.kicad_sch (KiCad schematic)
At the start: 28 parts, among them U1 STM32L475VGTx, X1 Not Fitted (NX3225GD-8.00M), X2 NX3215SA-32.768K

Commit message: Final report finished
Parts:
- C2, C4: footprint Capacitor_SMD:C_0402_1005Metric -> (none)
- R5, R7: footprint Resistor_SMD:R_0402_1005Metric -> (none)
Connections:
- net ARD.A1-ADC: no longer U1.34 (PC5)
- net ARD.A3-ADC: no longer U1.18 (PC3)
- net VDD: now also C8.1, SB17.2 (B), U1.6 (VBAT)
- net ISM43362-SPI3_CSN: no longer names the net of U1.97 (PE0)
- net LSM6DSL_INT1_EXTI11: no longer names the net of U1.58 (PD11)
- net M24SR64-Y-GPO: no longer names the net of U1.3 (PE4)
- net M24SR64-Y-RF_DISABLE: no longer names the net of U1.1 (PE2)
- net QUADSPI_BK1_IO0: no longer names the net of U1.43 (PE12)
- net QUADSPI_BK1_IO1: no longer names the net of U1.44 (PE13)
- net QUADSPI_BK1_IO2: no longer names the net of U1.45 (PE14)
- net QUADSPI_BK1_IO3: no longer names the net of U1.46 (PE15)
- net QUADSPI_NCS: no longer names the net of U1.42 (PE11)
- net SPBTLE-RF-SPI3_CSN: no longer names the net of U1.60 (PD13)
- net SPSGRF-915-SPI3_CSN: no longer names the net of U1.91 (PB5)
- net ST-LINK-UART1_RX: no longer names the net of U1.93 (PB7)
- net ST-LINK-UART1_TX: no longer names the net of U1.92 (PB6)
- net STSAFE-A100-RESET: no longer names the net of U1.88 (PD7)
- net SYS_JTMS-SWDIO: no longer names the net of U1.72 (PA13)
- net USB_OTG_FS_DM: no longer names the net of U1.70 (PA11)
- net USB_OTG_FS_DP: no longer names the net of U1.71 (PA12)
- net USB_OTG_FS_ID: no longer names the net of U1.69 (PA10)
- net USB_OTG_FS_OVRCR_EXTI3: no longer names the net of U1.2 (PE3)
- net USB_OTG_FS_PWR_EN: no longer names the net of U1.59 (PD12)
- net USB_OTG_FS_VBUS: no longer names the net of U1.68 (PA9)
- new net ARD.A0-ADC: U1.34 (PC5)
- new net ARD.A2-ADC: U1.18 (PC3)
