File: Embedded Systems Hardware Design/Project_HC/P3_Sensors.kicad_sch (KiCad schematic)
At the start: 10 parts, among them U10 Mic, U2 Mic

Commit message: HW5 finished
Parts:
- added C18, C21, C30: 4.7uF, Capacitor_SMD:C_0603_1608Metric, symbol Device:C
- added C19, C20, C22, C23, C25, C26, C28, C29, C31: 100nF, Capacitor_SMD:C_0402_1005Metric, symbol Device:C
- added C24: 1uF, Capacitor_SMD:C_0402_1005Metric, symbol Device:C
- added C27: 2.2uF, Capacitor_SMD:C_0603_1608Metric, symbol Device:C
- added R14: 10k, Resistor_SMD:R_0402_1005Metric, symbol Device:R
- added R15: 10K, Resistor_SMD:R_0402_1005Metric, symbol Device:R
- added U4: VL53L0X, VL53L0X:SENSOR_VL53L0X, symbol VL53L0X:VL53L0X
- added U5: LIS3MDL, Package_LGA:LGA-12_2x2mm_P0.5mm, symbol Sensor_Magnetic:LIS3MDL
- added U6: HTS221, XDCR_HTS221, symbol HTS221:HTS221
- added U7: LPS22HB, LPS22HB:LGA10R50P2X3_200X200X80, symbol Sensor_Pressure:LPS25HB
- C16, C17, C74: footprint (none) -> Capacitor_SMD:C_0603_1608Metric
- C46: footprint (none) -> Capacitor_SMD:C_0402_1005Metric
- R13, R6, R67: footprint (none) -> Resistor_SMD:R_0402_1005Metric
- gave numbers to parts that had none: 1
Connections:
- net +3.3V: now also C21.1, C22.1, C27.1, C28.1, U4.1 (AVDDVCSEL), U4.11 (AVDD), U6.1 (VDD), U6.6 (CS)
- net GND: now also U3.1 (SDO/SA0), U3.6 (GND), U3.7 (GND), C18.2, C19.2, C20.2, C21.2, C22.2, C23.2, C24.2, C25.2, C26.2, C27.2, C28.2, C29.2, C30.2, C31.2, U4.12 (GND), U4.2 (AVSSVCSEL), U4.3 (GND), U4.4 (GND), U4.6 (GND), U5.12 (Res), U5.2 (Res), U5.3 (GND), U6.5 (GND)
- net +3V3: now reaches U3.12 (CS)
- net +3V3: now also U3.5 (VDDIO), U3.8 (VDD), C18.1, C19.1, C20.1, C24.1, C25.1, C26.1, C29.1, C30.1, C31.1, R14.2, R15.2, U5.10 (~{CS}), U5.5 (Vdd), U5.6 (Vdd_IO), U5.9 (SDO/SA1), U7.1 (VDD_IO), U7.10 (VDD), U7.5 (SD0/SA0), U7.6 (~{CS})
- net INTERNAL-I2C2_SCL: now reaches U3.13 (SCL)
- net INTERNAL-I2C2_SCL: now also U4.10 (SCL), U5.1 (SCL/SPC), U6.2 (SCL/SPC), U7.2 (SCL/SPC)
- net INTERNAL-I2C2_SDA: now reaches U3.14 (SDA)
- net INTERNAL-I2C2_SDA: now also U3.4 (INT1), U4.9 (SDA), U5.11 (SDA/SDI/SDO), U6.4 (SDA/SDI/SDO), U7.4 (SDA/SDI/SDO)
- new net: C23.1, U5.4 (C1)
- new net GNDREF: U7.3 (RES), U7.8 (GND), U7.9 (GND)
- new net HTS221_DRDY_EXTI15: U6.3 (DRDY)
- new net LPS22HB_INT_DRDY_EXTI10: U7.7 (INT_DRDY)
- new net LSM3MDL_DRDY_EXTI8: U5.8 (DRDY)
- new net VL53L0X_GPIO1_EXTI7: R14.1, U4.7 (GPIO1)
- new net VL53L0X_XSHUT: R15.1, U4.5 (~{XSHUT})
Other:
- note added: "Accelerometer & Gyro"
- note added: "Barometer"
- note added: "Magnetometer"
- note added: "Microphone MEMS"
- note added: "Read=00111101 (3Dh) Write=00111100 (3Ch)"
- note added: "Read=01010011(53h) Write=01010010(52h)"
- note added: "Read=10111011 (BBh) Write=10111010 (BAh)"
- note added: "Read=10111111 (BFh) Write=10111110 (BEh)"
- note added: "Read=11010101 (D5h) Write=11010100 (D4h)"
- note added: "Temp & Humidity"

Commit message: Final report finished
Parts:
- C16: renamed from C17; value 0.1uF -> 100nF; footprint Capacitor_SMD:C_0603_1608Metric -> Capacitor_SMD:C_0402_1005Metric
- C21: renamed from C74; value 0.1uF -> 100nF; footprint Capacitor_SMD:C_0603_1608Metric -> Capacitor_SMD:C_0402_1005Metric
- C22: renamed from C46; footprint Capacitor_SMD:C_0402_1005Metric -> Capacitor_SMD:C_0603_1608Metric
- renumbered C16 to C17, C21 to C27, C22 to C28, C27 to C29, C28 to C30, C29 to C31, C30 to C32, C31 to C33, R6 to R1, R14 to R13, R15 to R14, R13 to R4, R67 to R6, U10 to U4, U4 to U6, U6 to U8
Connections:
- net GNDREF is gone; now on net GND: U7.3 (RES), U7.8 (GND), U7.9 (GND)
