File: Embedded Systems Hardware Design/Project_HC/P4_RF_Modules.kicad_sch (KiCad schematic)
At the start: 0 parts

Commit message: Final report finished
Parts:
- added C43, C44, C45: 100nF, Capacitor_SMD:C_0402_1005Metric, symbol Device:C
- added C47: 2.2uF, Capacitor_SMD:C_0402_1005Metric, symbol Device:C
- added C49, C50: 10uF, Capacitor_SMD:C_0603_1608Metric, symbol Device:C
- added C75, C76: 2.2uF, Capacitor_SMD:C_0603_1608Metric, symbol Device:C
- added M1: BT Module, RF_Module:ST_SPBTLE, symbol RF_Bluetooth:SPBTLE-RF
- added M2: ISM43362-M3G-L44, ISM43362-M3G-L44:INVENTEK_ISM43362-M3G-L44-E_C2.5.0.3_SPI, symbol ISM43362-M3G-L44-E_C2.5.0.3_SPI:ISM43362-M3G-L44-E_C2.5.0.3_SPI
- added M3: SPSGRF, SPSGRF-868:XCVR_SPSGRF-868, symbol SPSGRF-868:SPSGRF-868
- added R26: 47K, Resistor_SMD:R_0402_1005Metric, symbol Device:R
- added R64, R65, R66: Not Fitted (10k), Resistor_SMD:R_0402_1005Metric, symbol Device:R
- added TP1, TP2, TP3, TP4, TP5: TestPoint_Small, TestPoint:TestPoint_2Pads_Pitch2.54mm_Drill0.8mm, symbol Connector:TestPoint_Small
- added U12: LT1963EST-3.3, LT1963EST-3:SOT230P700X180-4N, symbol Regulator_Linear:LT1963AxST-3.3
Connections:
- new net: M2.6 (TDI), TP3.1
- new net: M2.7 (TDO), TP4.1
- new net: M2.28 (CFG0), R66.1
- new net: M2.29 (CFG1), R64.1, R65.1
- new net: M2.4 (TMS), TP1.1
- new net: M2.5 (TCK), TP2.1
- new net: M2.8 (TDRSTN), TP5.1
- new net +3V3: C43.1, C44.1, C45.1, C47.1, C50.1, C75.1, C76.1, M1.5 (VIN), M2.14 (VDD), M2.15 (VBAT), M2.2 (VDD), M3.5 (VIN), R26.2, R64.2, R65.2, R66.2, U12.3 (OUT)
- new net +5V: C49.1, U12.1 (IN)
- new net GND: C43.2, C44.2, C45.2, C47.2, C49.2, C50.2, C75.2, C76.2, M1.6 (GND), M2.1 (GND), M2.17 (GND), M2.20 (GND), M2.3 (GND), M2.35 (GND), M3.6 (GND), U12.2 (GND)
- new net INTERNAL-SPI3_MISO: M1.8 (SPI_MISO), M2.10 (ADC3/SPI_MISO), M3.8 (SPI_MISO)
- new net INTERNAL-SPI3_MOSI: M1.9 (SPI_MOSI), M2.9 (ADC4/SPI_MOSI), M3.9 (SPI_MOSI)
- new net INTERNAL-SPI3_SCK: M1.7 (SPI_CLK), M2.11 (ADC2/SPI_SCK), M3.7 (SPI_CLK)
- new net INTERNAL-UART3_RX: M2.22 (TX)
- new net INTERNAL-UART3_TX: M2.21 (RX)
- new net ISM43362-BOOT0: M2.33 (BOOT0/RES4)
- new net ISM43362-DRDY_EXTI1: M2.13 (ADC0/DATARDY)
- new net ISM43362-RST: M2.34 (RSTN)
- new net ISM43362-WAKEUP: M2.16 (WKUP)
- new net SPBTLE-RF-IRQ_EXTI6: M1.4 (SPI_IRQ)
- new net SPBTLE-RF-RST: M1.11 (~{BT_RESET})
- new net SPBTLE-RF-SPI3-CSN: M1.10 (SPI_~{CS}), M2.12 (ADC1/SPI_SSN), M3.10 (SPI_CS), R26.1
- new net SPSGRF-915-GPIO3_EXTI5: M3.1 (GPIO[3])
- new net SPSGRF-915-SDN: M3.11 (SDN)
