File: Embedded Systems Hardware Design/Project_HC/P5_Connectors.kicad_sch (KiCad schematic)
At the start: 25 parts, among them CN1 Header 10X1_Female_SMD, CN10 HEADER_2X6_PMOD, CN2 Header 8X1_Female_SMD, CN3 Header 8X1_Female_SMD, CN4 Header 6X1_Female_SMD, CN5 TC2050-IDC-NL

Commit message: Final report finished
Parts:
- removed SB5, SB6, SB7, SB8: Close, Jumper:SolderJumper-2_P1.3mm_Bridged2Bar_Pad1.0x1.5mm, symbol Jumper:SolderJumper_2_Bridged
- renumbered CN10 to CN6
Connections:
- net ARD0D130SPI10SCK0LED renamed ARD.D13-SPI1_SCK/LED1
- net ARD0D150I2C10 renamed ARD.D15-I2C1_SCL
- net ARD0D90P renamed ARD.D9-PWM
- new net: CN6.2 (Pin_2), SB12. (B), SB15. (B)
- new net: CN6.1 (Pin_1), SB14. (B), SB19. (B)
- new net: CN6.3 (Pin_3), SB18. (B), SB20. (B)
- new net: CN6.4 (Pin_4), SB16. (B), SB21. (B)
Other:
- note added: "TAG NRST"
- note added: "TAG SWCLK"
- note added: "TAG SWDIO"
- note added: "TAG SWO"
- note added: "T_JTCK"
- note added: "T_JTMS"
- note added: "T_NRST"
- note added: "T_SWO"
