File: Embedded Systems Hardware Design/Project_HC/P6_Mix.kicad_sch (KiCad schematic)
At the start: 0 parts

Commit message: HW5 finished
Parts:
- added B1: SW-PUSH-CMS_BLACK, Button_Switch_SMD:SW_Push_1P1T-MP_NO_Horizontal_Alps_SKRTLAE010, symbol Switch:SW_Push
- added B2: SW-PUSH-CMS_BLUE, Button_Switch_SMD:SW_Push_1P1T-MP_NO_Horizontal_Alps_SKRTLAE010, symbol Switch:SW_Push
- added C34, C36, C42, C73: 100nF, Capacitor_SMD:C_0402_1005Metric, symbol Device:C
- added C35, C37: 10pF, Capacitor_SMD:C_0402_1005Metric, symbol Device:C
- added C38, C39, C40, C41: 10uF, Capacitor_SMD:C_0603_1608Metric, symbol Device:C
- added HW1, HW2, HW3, HW4: SHUNT_BK, SNT-100-BK-G:Samtec-SNT-100-BK-G-MFG, symbol Graphic:Logo_Open_Hardware_Small
- added JP4: HEADER_2X5, Connector_PinHeader_2.54mm:PinHeader_2x05_P2.54mm_Horizontal, symbol Connector_Generic:Conn_02x05_Odd_Even
- added JP5, JP6, JP7: TSW-102-07-G-S, TSW-102-07-G-S:SAMTEC_TSW-102-07-G-S, symbol TSW-102-07-G-S:TSW-102-07-G-S
- added LD1, LD2, LD5: LED GREEN, LED_SMD:LED_0603_1608Metric, symbol Device:LED_Small_Filled
- added LD3: LED YELLOW, LED_SMD:LED_0603_1608Metric, symbol Device:LED_Small_Filled
- added LD4: LED BLUE, LED_SMD:LED_0603_1608Metric, symbol Device:LED_Small_Filled
- added R16: 10K, Resistor_SMD:R_0402_1005Metric, symbol Device:R
- added R18, R19, R21, R24: 1K, Resistor_SMD:R_0402_1005Metric, symbol Device:R
- added R20, R25: 330R, Resistor_SMD:R_0402_1005Metric, symbol Device:R
- added R22: 680R, Resistor_SMD:R_0402_1005Metric, symbol Device:R
- added R23: 100k, Resistor_SMD:R_0402_1005Metric, symbol Device:R
- added R38: 200k, Resistor_SMD:R_0402_1005Metric, symbol Device:R
- added SB1, SB2, SB3, SB4: Close, Jumper:SolderJumper-2_P1.3mm_Bridged2Bar_Pad1.0x1.5mm, symbol Jumper:SolderJumper_2_Bridged
- added U13: LD1117S50TR, Package_TO_SOT_SMD:SOT-223-3_TabPin2, symbol Regulator_Linear:LD1117S50TR_SOT223
- added U14: LD1117S33TR, Package_TO_SOT_SMD:SOT-223-3_TabPin2, symbol Regulator_Linear:LD1117S33TR_SOT223
- added U21: TSV631AILT, TSV631AILT:SOT95P280X145-5N, symbol Amplifier_Operational:LMV601
Connections:
- new net: C34.1, R19.2, SB2. (B)
- new net: LD3.2 (A), R21.1
- new net: B2.1, C37.1, R23.1, R24.1
- new net: LD5.2 (A), R25.1
- new net: B1.1, C35.1, R19.1
- new net: LD4.2 (A), R22.1
- new net: C36.1, R24.2, SB3. (B)
- new net: LD1.2 (A), R18.1
- new net: R18.2, U21.3 (-), U21.4
- new net: R16.1, R38.1, U21.1 (+)
- new net: LD2.2 (A), R20.1
- new net: R16.2, SB1. (B)
- new net +3.3V: C73.1, R23.2, U21.5 (V+)
- new net +3V3: C42.1, JP5.01, JP5.02, SB4. (B)
- new net +5V: C38.1, C39.1, C40.1, C41.1, JP4.1 (Pin_1), JP4.10 (Pin_10), JP4.2 (Pin_2), JP4.3 (Pin_3), JP4.4 (Pin_4), JP4.5 (Pin_5), JP4.6 (Pin_6), JP4.8 (Pin_8), JP4.9 (Pin_9), R25.2, SB4. (B), U13.2 (VO), U13.3 (VI), U14.2 (VO), U14.3 (VI), U14.4 (Tab)
- new net 5V_VBAT: JP4.7 (Pin_7)
- new net ARD.D13-SPI1_SCK/LED1: SB1. (B)
- new net BUTTON_EXTI13: SB3. (B)
- new net GND: B1.2, B2.2, C34.2, C35.2, C36.2, C37.2, C38.2, C39.2, C40.2, C41.2, C42.2, C73.2, JP6.01, JP6.02, JP7.01, JP7.02, LD1.1 (K), LD2.1 (K), LD3.1 (K), LD4.1 (K), LD5.1 (K), R38.2, U13.1 (GND), U14.1 (GND), U21.2 (V-)
- new net LED2: R20.2
- new net LED3(WIFI) & LED4(BLE): R21.2, R22.2
- new net STM_NRST: SB2. (B)
Other:
- note added: "100nF should be place close to the MCU 10pF and 1K should be place close to the button"
- note added: "3V3 / 800mA"
- note added: "3V3 PWR"
- note added: "5V / 800mA"
- note added: "5V INPUT PWR FROM ARDUINO"
- note added: "5V PWR SELECTION FROM EXTERNAL SOURCES"
- note added: "From Arduino power pin"
- note added: "GND PROBE"
- note added: "IDD"
- note added: "Jumper to measure IDD of the MCU"
- note added: "Open solder bridge if Discovery is supplied from +3V3 of extension connector"
- note added: "RESET BUTTON"
- note added: "The 2 LEDs are top side"
- note added: "USER & WAKE-UP Button"
- note added: "USER LED"

Commit message: Final report finished
Parts:
- B1: renamed from B2; footprint Button_Switch_SMD:SW_Push_1P1T-MP_NO_Horizontal_Alps_SKRTLAE010 -> Button_Switch_SMD:SW_DIP_SPSTx02_Slide_Copal_CHS-02B_W7.62mm_P1.27mm
- B2: renamed from B1; footprint Button_Switch_SMD:SW_Push_1P1T-MP_NO_Horizontal_Alps_SKRTLAE010 -> Button_Switch_SMD:SW_DIP_SPSTx02_Slide_Copal_CHS-02B_W7.62mm_P1.27mm
- C37: footprint Capacitor_SMD:C_0402_1005Metric -> Capacitor_SMD:C_0603_1608Metric
- renumbered HW3 to HW2, HW4 to HW3, HW2 to HW4, LD5 to LD1, LD1 to LD2, LD2 to LD3, LD3 to LD4, LD4 to LD5, U21 to U10
Connections:
- net 5V_VBAT: no longer names the net of JP4.7 (Pin_7)
Other:
- note added: "5V_VBAT"
